Commit message: Correction of errors in gazebo all packages

File: onrobot_2f/onrobot_description/urdf/gripper.urdf (robot description, URDF)
Before this commit: robot gripper_2f, 3 links, 2 joints
Links:
- link base_gripper: geometry collision mesh filename=package://onrobot_description/meshes/gripper_body.dae; visual mesh filename=package://onrobot_description/meshes/gripper_body.dae

File: robotiq_85_gripper/robotiq_85_description/urdf/robotiq_85_gripper.urdf.xacro (robot description, xacro)
@@ -299,5 +299,5 @@
             <kd>1.0</kd>
         </gazebo>
-	<gazebo>
+	<!--gazebo>
 	  <plugin name="gazebo_grasp_fix" filename="libgazebo_grasp_fix.so">
             <arm>
@@ -315,5 +315,5 @@
 	    <contact_topic>__default_topic__</contact_topic>
 	  </plugin>
-	</gazebo>
+	</gazebo-->
         <xacro:robotiq_85_gripper_transmission prefix="${prefix}" />
     </xacro:macro>

File: ur_gripper_sim/urdf/robot_gripper.xacro (robot description, xacro)
@@ -2,7 +2,7 @@
 <robot xmlns:xacro="http://ros.org/wiki/xacro" name="robot_gripper">
     <xacro:include filename="$(find ur_e_description)/urdf/ur3e_robot.urdf.xacro" />
-    <xacro:include filename="$(find my_gripper_description)/urdf/gripper.urdf" />
+    <xacro:include filename="$(find onrobot_description)/urdf/gripper.urdf" />
     <joint name="gipper_tool_joint" type="fixed">
-        <parent link="ee_link" />
+        <parent link="tool0" />
         <child link = "base_gripper" />
         <origin xyz="0.0 0.0 0.0" rpy="1.570 0.0 0.0" />

File: ur_gripper_sim/urdf/ur5_robotiq_gripper.xacro (robot description, xacro)
@@ -1,6 +1,5 @@
 <?xml version="1.0"?>
 <robot xmlns:xacro="http://ros.org/wiki/xacro" name="robot_gripper">
-     <xacro:include filename="$(find ur_e_description)/urdf/ur5e.urdf.xacro" />
-     <xacro:ur5e_robot prefix="" joint_limited="false"/>
+     <xacro:include filename="$(find ur_e_description)/urdf/ur5e_robot.urdf.xacro" />
      <!-- robotiq 85 -->
     <xacro:include filename="$(find robotiq_85_description)/urdf/robotiq_85_gripper.urdf.xacro" />
