Commit message: modifications for getting right gazebo simulations in ur5 ur3

File: ur_gripper_sim/urdf/ur5_robotiq_gripper.xacro (robot description, xacro)
@@ -1,5 +1,10 @@
 <?xml version="1.0"?>
 <robot xmlns:xacro="http://ros.org/wiki/xacro" name="robot_gripper">
-     <xacro:include filename="$(find ur_e_description)/urdf/ur5e_robot.urdf.xacro" />
+      <!-- common stuff -->
+  <xacro:include filename="$(find ur_e_description)/urdf/common.gazebo.xacro" />
+  <!-- ur5e -->
+  <xacro:include filename="$(find ur_e_description)/urdf/ur5e.urdf.xacro" />
+  <!-- arm -->
+  <xacro:ur5e_robot prefix="" joint_limited="false"/>
      <!-- robotiq 85 -->
     <xacro:include filename="$(find robotiq_85_description)/urdf/robotiq_85_gripper.urdf.xacro" />
@@ -8,3 +13,9 @@
       <origin xyz="0 0 0" rpy="0 0 0"/>
     </xacro:robotiq_85_gripper>
+  <link name="world" />
+  <joint name="world_joint" type="fixed">
+    <parent link="world" />
+    <child link = "base_link" />
+    <origin xyz="0.0 0.0 0.0" rpy="0.0 0.0 0.0" />
+  </joint>
 </robot>
