Commit message: Cambios en paquetes UR gripper, tutorial moveit

File: ur_gripper_sim/urdf/ur5_robotiq_gripper.urdf.xacro (robot description, xacro)
@@ -1,5 +1,5 @@
 <?xml version="1.0"?>
 <robot xmlns:xacro="http://ros.org/wiki/xacro" name="robot_gripper">
-      <!-- common stuff -->
+  <!-- common stuff -->
   <xacro:include filename="$(find ur_e_description)/urdf/common.gazebo.xacro" />
   <!-- ur5e -->
@@ -7,9 +7,9 @@
   <!-- arm -->
   <xacro:ur5e_robot prefix="" joint_limited="false"/>
-     <!-- robotiq 85 -->
-    <xacro:include filename="$(find robotiq_85_description)/urdf/robotiq_85_gripper.urdf.xacro" />
-    <!-- gripper -->
-    <xacro:robotiq_85_gripper prefix="" parent="ee_link" >
-      <origin xyz="0 0 0" rpy="0 0 0"/>
-    </xacro:robotiq_85_gripper>
+  <!-- robotiq 85 -->
+  <xacro:include filename="$(find robotiq_85_description)/urdf/robotiq_85_gripper.urdf.xacro" />
+  <!-- gripper -->
+  <xacro:robotiq_85_gripper prefix="" parent="ee_link" >
+    <origin xyz="0 0 0" rpy="0 0 0"/>
+  </xacro:robotiq_85_gripper>
 </robot>

File: ur_gripper_sim/urdf/ur5_robotiq_gripper.xacro (robot description, xacro)
@@ -1,5 +1,5 @@
 <?xml version="1.0"?>
 <robot xmlns:xacro="http://ros.org/wiki/xacro" name="robot_gripper">
-      <!-- common stuff -->
+  <!-- common stuff -->
   <xacro:include filename="$(find ur_e_description)/urdf/common.gazebo.xacro" />
   <!-- ur5e -->
@@ -7,10 +7,10 @@
   <!-- arm -->
   <xacro:ur5e_robot prefix="" joint_limited="false"/>
-     <!-- robotiq 85 -->
-    <xacro:include filename="$(find robotiq_85_description)/urdf/robotiq_85_gripper.urdf.xacro" />
-    <!-- gripper -->
-    <xacro:robotiq_85_gripper prefix="" parent="ee_link" >
-      <origin xyz="0 0 0" rpy="0 0 0"/>
-    </xacro:robotiq_85_gripper>
+  <!-- robotiq 85 -->
+  <xacro:include filename="$(find robotiq_85_description)/urdf/robotiq_85_gripper.urdf.xacro" />
+  <!-- gripper -->
+  <xacro:robotiq_85_gripper prefix="" parent="ee_link" >
+    <origin xyz="0 0 0" rpy="0 0 0"/>
+  </xacro:robotiq_85_gripper>
   <link name="world" />
   <joint name="world_joint" type="fixed">
