Commit message: updated packages

File: robotiq_85_gripper/robotiq_85_description/urdf/robotiq_85_gripper.transmission.xacro (robot description, xacro)
@@ -12,37 +12,4 @@
             </actuator>
         </transmission>
-        <gazebo>
-                <!-- loading plugin: mimic joints works in gazebo now -->
-            <plugin filename="libroboticsgroup_gazebo_mimic_joint_plugin.so" name="${prefix}mimic_robotiq_85_1">
-                <joint>${prefix}gripper_finger1_joint</joint>
-                <mimicJoint>${prefix}gripper_finger2_joint</mimicJoint>
-                <!--multiplier>1.0</multiplier>
-                <offset>0.0</offset-->
-            </plugin>
-            <plugin filename="libroboticsgroup_gazebo_mimic_joint_plugin.so" name="${prefix}mimic_robotiq_85_2">
-                <joint>${prefix}gripper_finger1_joint</joint>
-                <mimicJoint>${prefix}gripper_finger2_inner_knuckle_joint</mimicJoint>
-                <!--multiplier>1.0</multiplier>
-                <offset>0.0</offset-->
-            </plugin>
-            <plugin filename="libroboticsgroup_gazebo_mimic_joint_plugin.so" name="${prefix}mimic_robotiq_85_3">
-                <joint>${prefix}gripper_finger1_joint</joint>
-                <mimicJoint>${prefix}gripper_finger1_inner_knuckle_joint</mimicJoint>
-                <!--multiplier>1.0</multiplier>
-                <offset>0.0</offset-->
-            </plugin>
-            <plugin filename="libroboticsgroup_gazebo_mimic_joint_plugin.so" name="${prefix}mimic_robotiq_85_4">
-                <joint>${prefix}gripper_finger1_joint</joint>
-                <mimicJoint>${prefix}gripper_finger1_finger_tip_joint</mimicJoint>
-                <multiplier>-1.0</multiplier>
-                <offset>0.0</offset>
-            </plugin>
-            <plugin filename="libroboticsgroup_gazebo_mimic_joint_plugin.so" name="${prefix}mimic_robotiq_85_5">
-                <joint>${prefix}gripper_finger1_joint</joint>
-                <mimicJoint>${prefix}gripper_finger2_finger_tip_joint</mimicJoint>
-                <multiplier>-1.0</multiplier>
-                <offset>0.0</offset>
-            </plugin>
-        </gazebo>
     </xacro:macro>
 </robot>

File: robotiq_85_gripper/robotiq_85_description/urdf/robotiq_85_gripper.urdf.xacro (robot description, xacro)
@@ -299,22 +299,7 @@
             <kd>1.0</kd>
         </gazebo>
-	<!--gazebo>
-	  <plugin name="gazebo_grasp_fix" filename="libgazebo_grasp_fix.so">
-            <arm>
-              <arm_name>gripper_arm</arm_name>
-              <palm_link>${parent}</palm_link>
-              <gripper_link>${prefix}gripper_finger1_finger_tip_link</gripper_link>
-              <gripper_link>${prefix}gripper_finger2_finger_tip_link</gripper_link>
-            </arm>
-	    <forces_angle_tolerance>100</forces_angle_tolerance>
-	    <update_rate>2</update_rate>
-	    <grip_count_threshold>1</grip_count_threshold>
-	    <max_grip_count>2</max_grip_count>
-	    <release_tolerance>0.005</release_tolerance>
-	    <disable_collisions_on_attach>true</disable_collisions_on_attach>
-	    <contact_topic>__default_topic__</contact_topic>
-	  </plugin>
-	</gazebo-->
         <xacro:robotiq_85_gripper_transmission prefix="${prefix}" />
     </xacro:macro>
+      <xacro:include filename="$(find robotiq_85_description)/urdf/gazebo_grasp.xacro" />
+    <xacro:include filename="$(find robotiq_85_description)/urdf/gazebo_mimic.xacro" />
 </robot>

File: ur_gripper_sim/urdf/ur5_robotiq_gripper.urdf.xacro (robot description, xacro)
@@ -13,3 +13,17 @@
       <origin xyz="0 0 0" rpy="0 0 0"/>
     </xacro:robotiq_85_gripper>
+   <link name="world" />
+  <joint name="world_joint" type="fixed">
+    <parent link="world" />
+    <child link = "base_link" />
+    <origin xyz="0.0 0.0 0.0" rpy="0.0 0.0 0.0" />
+  </joint>
+  <xacro:include filename="$(find kinect_v2)/urdf/kinect_v2.urdf.xacro" />
+     <!--link name="world"/-->
+    <xacro:kinect_v2  parent="world">
+        <origin xyz="0.4 0 1.2"
+                rpy="0 1.57 0" />
+    </xacro:kinect_v2>
+    <xacro:include filename="$(find ur_gripper_sim)/urdf/gazebo_grasp.xacro" />
+    <xacro:include filename="$(find ur_gripper_sim)/urdf/gazebo_mimic.xacro" />
 </robot>

File: ur_gripper_sim/urdf/ur5_robotiq_gripper.xacro (robot description, xacro)
@@ -13,4 +13,10 @@
       <origin xyz="0 0 0" rpy="0 0 0"/>
     </xacro:robotiq_85_gripper>
+      <xacro:include filename="$(find kinect_v2)/urdf/kinect_v2.urdf.xacro" />
+     <!--link name="world"/-->
+    <xacro:kinect_v2  parent="world">
+        <origin xyz="0.4 0 1.2"
+                rpy="0 1.57 0" />
+    </xacro:kinect_v2>
   <link name="world" />
   <joint name="world_joint" type="fixed">
