Commit message: multicrontrol in gazebo ofr multirobot system

File: robot_cell/cell_description/urdf/cell_integration.xacro (robot description, xacro)
@@ -1,17 +1,29 @@
 <?xml version="1.0"?>
 <robot xmlns:xacro="http://ros.org/wiki/xacro" name="robot_gripper">
-    <xacro:include filename="$(find ur_gripper_sim)/urdf/ur5_robotiq_gripper.xacro" />
-    <xacro:include filename="$(find mesa_general)/urdf/mesa_general.urdf" />
+       <xacro:include filename="$(find mesa_general)/urdf/mesa_general.urdf" />
     <xacro:include filename="$(find mesa_general)/urdf/objects/block.urdf" />
     <joint name="mesa_block_joint" type="fixed">
-        <parent link="mesa_base_link" />
+        <parent link="world" />
         <child link = "block" />
-        <origin xyz="0.6 -0.3 0.99" rpy="0.0 0.0 0.0" />
+        <origin xyz="0.5 -0.3 0.92" rpy="0.0 0.0 0.0" />
       </joint>
-    <joint name="mesa_robot_joint" type="fixed">
-        <parent link="mesa_base_link" />
-        <child link = "base_link" />
-        <origin xyz="0.02 -0.220 0.99" rpy="0.0 0.0 -1.57" />
+    <xacro:include filename="$(find ur_gripper_sim)/urdf/ur5_robotiq_gripper.urdf.xacro" />
+    <joint name="mesa_robot1_joint" type="fixed">
+        <parent link="world" />
+        <child link = "r1base_link" />
+        <origin xyz="-0.1 -0.30 0.90" rpy="0.0 0.0 -1.57" />
       </joint>
+   <xacro:include filename="$(find ur_gripper_sim)/urdf/r2_ur3_onrobot_gripper.urdf.xacro" />
+    <joint name="mesa_robot2_joint" type="fixed">
+      <parent link="world" />
+      <child link = "r2base_link" />
+      <origin xyz="1.1 -0.30 0.90" rpy="0.0 0.0 -1.57" />
+    </joint>
+     <xacro:include filename="$(find ur_gripper_sim)/urdf/r3_ur3_onrobot_gripper.urdf.xacro" />
+    <joint name="mesa_robot3_joint" type="fixed">
+      <parent link="world" />
+      <child link = "r3base_link" />
+      <origin xyz="-1.1 -0.30 0.90" rpy="0.0 0.0 -1.57" />
+    </joint>
 <link name="world"/>
   <joint name="world_mesa" type="fixed">
@@ -20,7 +32,8 @@
       <origin xyz="0 0 0" rpy="0 0 0"/>
   </joint>
-   <gazebo>
-    <plugin filename="libgazebo_ros_control.so" name="gazebo_ros_control">
-      <robotNamesapce>/gripper_2fs</robotNamesapce>
+  <gazebo>
+    <plugin name="ros_control" filename="libgazebo_ros_control.so">
+      <!--robotNamespace>/</robotNamespace-->
+      <!--robotSimType>gazebo_ros_control/DefaultRobotHWSim</robotSimType-->
     </plugin>
   </gazebo>

File: robot_cell/mesa_general/urdf/mesa_general.urdf (robot description, URDF)
Before this commit: robot mesa_general, 1 links, 0 joints
Links:
- link mesa_base_link: geometry collision mesh filename=package://mesa_general/meshes/mesa_general.dae; visual mesh filename=package://mesa_general/meshes/mesa_general.dae

File: robot_cell/mesa_general/urdf/objects/block.urdf (robot description, URDF)
Before this commit: robot block, 1 links, 0 joints
Links:
- link block: geometry collision box size=0.04 0.04 0.04; visual box size=0.04 0.04 0.04

File: robotiq_85_gripper/robotiq_85_description/urdf/gazebo_grasp.xacro (robot description, xacro)
@@ -2,14 +2,15 @@
 <root  xmlns:xacro="http://ros.org/wiki/xacro">
     <!-- https://github.com/JenniferBuehler/gazebo-pkgs/wiki/The-Gazebo-grasp-fix-plugin -->
+<xacro:macro name="gazebo_grasp_plugin" params="prefix">
 <gazebo>
     <plugin name="gazebo_grasp_fix" filename="libgazebo_grasp_fix.so">
         <arm>
            <arm_name>ur5e_robot</arm_name>  <!-- name of this arm. Has to be unique.-->
-            <palm_link>gripper_finger1_inner_knuckle_link</palm_link>
+            <palm_link>${prefix}gripper_finger1_inner_knuckle_link</palm_link>
            <!--  has to be the link to which the finger joints are attached. -->
-            <gripper_link>gripper_finger2_inner_knuckle_link</gripper_link>
+            <gripper_link>${prefix}gripper_finger2_inner_knuckle_link</gripper_link>
            <!-- tags have to include all link names of the gripper/hand which are used to actively grasp objects -->
-              <gripper_link>gripper_finger1_finger_tip_link</gripper_link>
-              <gripper_link>gripper_finger2_finger_tip_link</gripper_link>
+              <gripper_link>${prefix}gripper_finger1_finger_tip_link</gripper_link>
+              <gripper_link>${prefix}gripper_finger2_finger_tip_link</gripper_link>
        </arm>
        <forces_angle_tolerance>100</forces_angle_tolerance>
@@ -22,3 +23,4 @@
     </plugin>
   </gazebo>
+  </xacro:macro>
 </root>

File: robotiq_85_gripper/robotiq_85_description/urdf/gazebo_mimic.xacro (robot description, xacro)
@@ -1,36 +1,38 @@
 <?xml version="1.0" encoding="UTF-8"?>
 <root xmlns:xacro="http://ros.org/wiki/xacro">
+<xacro:macro name="gazebo_mimic_plugin" params="prefix">
  <gazebo>
                 <!-- loading plugin: mimic joints works in gazebo now -->
             <plugin filename="libroboticsgroup_gazebo_mimic_joint_plugin.so" name="mimic_robotiq_85_1">
-                <joint>gripper_finger1_joint</joint>
-                <mimicJoint>gripper_finger2_joint</mimicJoint>
+                <joint>${prefix}gripper_finger1_joint</joint>
+                <mimicJoint>${prefix}gripper_finger2_joint</mimicJoint>
                 <!--multiplier>1.0</multiplier>
                 <offset>0.0</offset-->
             </plugin>
             <plugin filename="libroboticsgroup_gazebo_mimic_joint_plugin.so" name="mimic_robotiq_85_2">
-                <joint>gripper_finger1_joint</joint>
-                <mimicJoint>gripper_finger2_inner_knuckle_joint</mimicJoint>
+                <joint>${prefix}gripper_finger1_joint</joint>
+                <mimicJoint>${prefix}gripper_finger2_inner_knuckle_joint</mimicJoint>
                 <!--multiplier>1.0</multiplier>
                 <offset>0.0</offset-->
             </plugin>
             <plugin filename="libroboticsgroup_gazebo_mimic_joint_plugin.so" name="mimic_robotiq_85_3">
-                <joint>gripper_finger1_joint</joint>
-                <mimicJoint>gripper_finger1_inner_knuckle_joint</mimicJoint>
+                <joint>${prefix}gripper_finger1_joint</joint>
+                <mimicJoint>${prefix}gripper_finger1_inner_knuckle_joint</mimicJoint>
                 <!--multiplier>1.0</multiplier>
                 <offset>0.0</offset-->
             </plugin>
             <plugin filename="libroboticsgroup_gazebo_mimic_joint_plugin.so" name="mimic_robotiq_85_4">
-                <joint>gripper_finger1_joint</joint>
-                <mimicJoint>gripper_finger1_finger_tip_joint</mimicJoint>
+                <joint>${prefix}gripper_finger1_joint</joint>
+                <mimicJoint>${prefix}gripper_finger1_finger_tip_joint</mimicJoint>
                 <multiplier>-1.0</multiplier>
                 <offset>0.0</offset>
             </plugin>
             <plugin filename="libroboticsgroup_gazebo_mimic_joint_plugin.so" name="mimic_robotiq_85_5">
-                <joint>gripper_finger1_joint</joint>
-                <mimicJoint>gripper_finger2_finger_tip_joint</mimicJoint>
+                <joint>${prefix}gripper_finger1_joint</joint>
+                <mimicJoint>${prefix}gripper_finger2_finger_tip_joint</mimicJoint>
                 <multiplier>-1.0</multiplier>
                 <offset>0.0</offset>
             </plugin>
  </gazebo>
+ </xacro:macro>
 </root>

File: robotiq_85_gripper/robotiq_85_description/urdf/robotiq_85_gripper.transmission.xacro (robot description, xacro)
@@ -5,9 +5,9 @@
             <type>transmission_interface/SimpleTransmission</type>
             <joint name="${prefix}gripper_finger1_joint">
-                <hardwareInterface>PositionJointInterface</hardwareInterface>
+                <hardwareInterface>hardware_interface/PositionJointInterface</hardwareInterface>
             </joint>
             <actuator name="${prefix}gripper_finger1_motor">
                 <mechanicalReduction>1</mechanicalReduction>
-                <hardwareInterface>PositionJointInterface</hardwareInterface>
+                <hardwareInterface>hardware_interface/PositionJointInterface</hardwareInterface>
             </actuator>
         </transmission>

File: robotiq_85_gripper/robotiq_85_description/urdf/robotiq_85_gripper.urdf.xacro (robot description, xacro)
@@ -2,4 +2,6 @@
 <robot name="robotiq_85_gripper" xmlns:xacro="http://ros.org/wiki/xacro">
     <xacro:include filename="$(find robotiq_85_description)/urdf/robotiq_85_gripper.transmission.xacro" />
+    <xacro:include filename="$(find robotiq_85_description)/urdf/gazebo_grasp.xacro" />
+    <xacro:include filename="$(find robotiq_85_description)/urdf/gazebo_mimic.xacro" />
     <xacro:macro name="robotiq_85_gripper" params="prefix parent *origin">
         <joint name="${prefix}gripper_base_joint" type="fixed">
@@ -300,6 +302,6 @@
         </gazebo>
         <xacro:robotiq_85_gripper_transmission prefix="${prefix}" />
+        <xacro:gazebo_grasp_plugin prefix="${prefix}" />
+        <xacro:gazebo_mimic_plugin prefix="${prefix}" />
     </xacro:macro>
-      <xacro:include filename="$(find robotiq_85_description)/urdf/gazebo_grasp.xacro" />
-    <xacro:include filename="$(find robotiq_85_description)/urdf/gazebo_mimic.xacro" />
 </robot>

File: ur_gripper_sim/urdf/ur5_robotiq_gripper.urdf.xacro (robot description, xacro)
@@ -1,29 +1,19 @@
 <?xml version="1.0"?>
-<robot xmlns:xacro="http://ros.org/wiki/xacro" name="robot_gripper">
-      <!-- common stuff -->
-  <xacro:include filename="$(find ur_e_description)/urdf/common.gazebo.xacro" />
-  <!-- ur5e -->
+<robot xmlns:xacro="http://ros.org/wiki/xacro" name="ur5_robot_gripper">
+   <!-- ur5e -->
   <xacro:include filename="$(find ur_e_description)/urdf/ur5e.urdf.xacro" />
   <!-- arm -->
-  <xacro:ur5e_robot prefix="" joint_limited="false"/>
-     <!-- robotiq 85 -->
-    <xacro:include filename="$(find robotiq_85_description)/urdf/robotiq_85_gripper.urdf.xacro" />
-    <!-- gripper -->
-    <xacro:robotiq_85_gripper prefix="" parent="ee_link" >
-      <origin xyz="0 0 0" rpy="0 0 0"/>
-    </xacro:robotiq_85_gripper>
-   <link name="world" />
-  <joint name="world_joint" type="fixed">
-    <parent link="world" />
-    <child link = "base_link" />
-    <origin xyz="0.0 0.0 0.0" rpy="0.0 0.0 0.0" />
-  </joint>
-  <xacro:include filename="$(find kinect_v2)/urdf/kinect_v2.urdf.xacro" />
-     <!--link name="world"/-->
+  <xacro:ur5e_robot prefix="r1" joint_limited="false"/>
+ <!-- robotiq 85 -->
+  <xacro:include filename="$(find robotiq_85_description)/urdf/robotiq_85_gripper.urdf.xacro"/>
+  <!-- gripper -->
+  <xacro:robotiq_85_gripper prefix="r1" parent="r1ee_link" >
+    <origin xyz="0 0 0" rpy="0 0 0"/>
+  </xacro:robotiq_85_gripper>
+  <!--xacro:include filename="$(find kinect_v2)/urdf/kinect_v2.urdf.xacro" />
+     <link name="world"/>
     <xacro:kinect_v2  parent="world">
         <origin xyz="0.4 0 1.2"
                 rpy="0 1.57 0" />
-    </xacro:kinect_v2>
-    <xacro:include filename="$(find ur_gripper_sim)/urdf/gazebo_grasp.xacro" />
-    <xacro:include filename="$(find ur_gripper_sim)/urdf/gazebo_mimic.xacro" />
+    </xacro:kinect_v2-->
 </robot>

File: ur_gripper_sim/urdf/ur5_robotiq_gripper.xacro (robot description, xacro)
@@ -13,15 +13,15 @@
       <origin xyz="0 0 0" rpy="0 0 0"/>
     </xacro:robotiq_85_gripper>
-      <xacro:include filename="$(find kinect_v2)/urdf/kinect_v2.urdf.xacro" />
-     <!--link name="world"/-->
+      <!--xacro:include filename="$(find kinect_v2)/urdf/kinect_v2.urdf.xacro" />
+     <link name="world"/>
     <xacro:kinect_v2  parent="world">
         <origin xyz="0.4 0 1.2"
                 rpy="0 1.57 0" />
-    </xacro:kinect_v2>
+    </xacro:kinect_v2-->
   <link name="world" />
   <joint name="world_joint" type="fixed">
     <parent link="world" />
     <child link = "base_link" />
-    <origin xyz="0.0 0.0 0.0" rpy="0.0 0.0 0.0" />
+    <origin xyz="0.0 0.0 1.01" rpy="0.0 0.0 0.0" />
   </joint>
 </robot>
